Commit message: Add files via upload

File: src/mower_main/model/mower.urdf (robot description, URDF)
Before this commit: robot ardumower, 6 links, 5 joints
Links:
- removed link imu_link
- removed link laser_base
- removed link laser_link
- added link gps; visual box size=0.020 0.027 0.010
- added link imu; visual box size=0.020 0.027 0.010
Joints:
- removed joint base_to_laserbase
- removed joint base_to_laserlink
- added joint base_to_gps: type fixed, parent base_link, child gps, origin xyz=0 0.08 0.223 rpy=0 0 0
- joint base_to_imu: child imu_link -> imu; origin xyz=0 0 0.223 rpy=0 0 0 -> xyz=-0.405 0 0.223 rpy=0 0 0
